Commit message: Added Kinect RGBD to URDF and gazebo file.
Made changes to model to implement new depth camera in simulation.

Samira Wettasinghe

File: src/my_robot/urdf/my_robot.xacro (robot description, xacro)
@@ -176,3 +176,10 @@
 	<axis xyz="0 1 0" rpy="0 0 0"/>
   </joint>
+  <joint name="camera_optical_joint" type="fixed">
+    <origin xyz="0 0 0" rpy="-1.5707 0 -1.5707"/>
+    <parent link="camera_link"/>
+    <child link="camera_link_optical"/>
+  </joint>
+  <link name="camera_link_optical">
+  </link>
 </robot>
